File: hardware/project-esp32-c3-wroom-02-breakout.kicad_pcb (KiCad board)
At the start: 2 copper layers, 25.4 x 32 mm, 10 parts, among them IC1 ESP32-WROVER-E_M213EH6464PH3Q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, J1 Conn_01x06_Male, J2 Conn_01x10_Male, J3 Conn_01x10_Male, Q1 MUN5214DW1T1G, U1 XC6220B331MR

Commit message: First placement done
Parts:
- removed C3: 0.1uF, Capacitor_SMD:C_0603_1608Metric_Pad1.08x0.95mm_HandSolder
- removed IC1: ESP32-WROVER-E_M213EH6464PH3Q0_, ESP32-WROVER-E:ESP32WROVEREM213EH6464PH3Q0
- added C2: 0.1uF, Capacitor_SMD:C_0603_1608Metric_Pad1.08x0.95mm_HandSolder, F.Cu at (45.5, 55.6)
- added C5: 22pF, Capacitor_SMD:C_0603_1608Metric_Pad1.08x0.95mm_HandSolder, F.Cu at (57.9, 50.8)
- added C6: 22pF, Capacitor_SMD:C_0603_1608Metric_Pad1.08x0.95mm_HandSolder, F.Cu at (53.8, 50.8)
- added D1: LED, LED_SMD:LED_0603_1608Metric, F.Cu at (61.7, 56.4)
- added JP1: SolderJumper_3_Bridged12, Jumper:SolderJumper-3_P1.3mm_Bridged12_RoundedPad1.0x1.5mm, F.Cu at (42.2, 50.8)
- added R2: 10k, Resistor_SMD:R_0603_1608Metric_Pad0.98x0.95mm_HandSolder, F.Cu at (42.4, 55.6)
- added R3: 10k, Resistor_SMD:R_0603_1608Metric_Pad0.98x0.95mm_HandSolder, F.Cu at (40.9, 55.6)
- added R4: 4k7, Resistor_SMD:R_0603_1608Metric_Pad0.98x0.95mm_HandSolder, F.Cu at (53.8, 49.3)
- added R5: 4k7, Resistor_SMD:R_0603_1608Metric_Pad0.98x0.95mm_HandSolder, F.Cu at (57.9, 49.3)
- added R6: 10k, Resistor_SMD:R_0603_1608Metric_Pad0.98x0.95mm_HandSolder, F.Cu at (59.9, 56.5)
- added U2: ESP32-C3-WROOM-02-H4, ESP32-C3-WROOM-02-H4:MODULE_ESP32-C3-WROOM-02-H4, F.Cu at (50.0, 37.8)
- J1: value Conn_01x06_Male -> SM04B-SRSS-TB(LF)(SN); footprint B6B-ZR(LF)(SN):JST_B6B-ZR(LF)(SN) -> SM04B-SRSS-TB(LF)(SN):JST_SM04B-SRSS-TB(LF)(SN)
- J2, J3: value Conn_01x10_Male -> Conn_01x08_Male; footprint Connector_PinHeader_2.54mm:PinHeader_1x10_P2.54mm_Vertical -> Connector_PinHeader_2.54mm:PinHeader_1x08_P2.54mm_Vertical
- moved C1 13.0 mm to (45.0, 50.8)
- moved U1 12.8 mm to (47.8, 50.8)
- moved C4 12.7 mm to (50.5, 50.8), turned to 90 degrees
- moved J1 10.1 mm to (54.9, 53.1), turned to 0 degrees
- moved Q1 7.89 mm to (49.0, 55.6)
- moved R1 7.66 mm to (43.9, 55.6), turned to 90 degrees
Connections:
- C1 pad 1: +5V -> VCC
- J1 pad 1: +5V -> GND
- J1 pad 2: /TX -> Net-(J1-Pad2)
- J1 pad 3: /RX -> /SDA
- J1 pad 4: /DTR -> /SCL
- J2 pad 1: /RESET -> +3V3
- J2 pad 2: /GPIO32 -> /RESET
- J2 pad 3: /GPIO33 -> /GPIO4
- J2 pad 4: /GPIO25 -> /GPIO5
- J2 pad 5: /GPIO26 -> /GPIO6
- J2 pad 6: /GPIO27 -> /GPIO7
- J2 pad 7: /GPIO14 -> VCC
- J3 pad 1: GND -> /GPIO0
- J3 pad 2: /GPIO23 -> /GPIO1
- J3 pad 3: /GPIO22 -> /GPIO3
- J3 pad 4: /GPIO21 -> /RX
- J3 pad 5: /GPIO19 -> /TX
- J3 pad 6: /GPIO18 -> /DTR
- J3 pad 7: /GPIO5 -> /RTS
- J3 pad 8: /GPIO4 -> /GPIO10
- Q1 pad 3: /GPIO0 -> /GPIO9
- U1 pad 1: +5V -> VCC
- U1 pad 3: +5V -> VCC
Routing:
- net /RESET: track 43.5 -> 0.00 mm, vias 1 -> 0
- net GND: track 29.0 -> 0.00 mm, vias 13 -> 0
- net /TX: track 26.6 -> 0.00 mm
- net /RX: track 24.8 -> 0.00 mm
- net +5V: track 20.6 -> 0.00 mm
- net /GPIO0: track 19.7 -> 0.00 mm, vias 2 -> 0
- net /RTS: track 14.0 -> 0.00 mm
- net +3V3: track 13.7 -> 0.00 mm
- net /DTR: track 11.6 -> 0.00 mm
- net /GPIO32: track 7.32 -> 0.00 mm
- net /GPIO5: track 6.11 -> 0.00 mm
- net /GPIO15: track 6.11 -> 0.00 mm
- net /GPIO33: track 6.10 -> 0.00 mm
- net /GPIO2: track 5.13 -> 0.00 mm
- net /GPIO4: track 4.84 -> 0.00 mm
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- removed copper zone on F.Cu, net +3V3
- removed copper zone on F.Cu, net +5V
- removed copper zone on B.Cu, net GND
Other:
- board size 25.4 x 32 mm -> 25.4 x 24.4 mm
- copper layers 2 -> 4
- board text added: "0"
- board text added: "1"
- board text added: "3"
- board text added: "6"
- board text added: "7"
- board text added: "DTR"
- board text added: "RTS"
- board text added: "RX"
- board text added: "TX"
- board text added: "VCC"
- board text removed: "14"
- board text removed: "15"
- board text removed: "18"
- board text removed: "19"
- board text removed: "2"
- board text removed: "21"
- board text removed: "22"
- board text removed: "23"
- board text removed: "25"
- board text removed: "26"
- board text removed: "27"
- board text removed: "32"
- board text removed: "33"
- board text removed: "5V"

Commit message: Routing done
Parts:
- moved JP1 8.13 mm to (50.3, 51.0)
- moved C5 4.06 mm to (53.8, 50.8), turned to 180 degrees
- moved R5 4.06 mm to (53.8, 49.3), turned to 0 degrees
- moved C6 3.56 mm to (57.4, 50.8), turned to 0 degrees
- moved R4 3.56 mm to (57.4, 49.3), turned to 180 degrees
- moved C1 3.05 mm to (41.9, 50.8)
- moved C4 3.05 mm to (47.5, 50.8)
- moved U1 3.05 mm to (44.7, 50.8)
Connections:
- C5 pad 1: /SCL -> /USB_D+
- C6 pad 1: /SDA -> /USB_D-
- J1 pad 3: /SDA -> /USB_D+
- J1 pad 4: /SCL -> /USB_D-
- J3 pad 4: /RX -> /TX
- J3 pad 5: /TX -> /RX
- R4 pad 2: /SDA -> /USB_D-
- R5 pad 2: /SCL -> /USB_D+
- U2 pad 13: /SDA -> /USB_D-
- U2 pad 14: /SCL -> /USB_D+
Routing:
- net /GPIO2: track 0.00 -> 30.3 mm, vias 0 -> 2
- net /RESET: track 0.00 -> 29.4 mm, vias 0 -> 2
- net GND: track 0.00 -> 24.3 mm, vias 0 -> 11
- net /DTR: track 0.00 -> 19.7 mm, vias 0 -> 1
- net /GPIO9: track 0.00 -> 19.4 mm, vias 0 -> 2
- net /RTS: track 0.00 -> 19.0 mm, vias 0 -> 1
- net +3V3: track 0.00 -> 17.3 mm, vias 0 -> 5
- net /GPIO8: track 0.00 -> 16.2 mm, vias 0 -> 2
- net /USB_D+: track 0.00 -> 14.3 mm
- net /USB_D-: track 0.00 -> 12.8 mm
- net Net-(J1-Pad2): track 0.00 -> 9.11 mm
- net /GPIO7: track 0.00 -> 8.84 mm, vias 0 -> 1
- net /GPIO10: track 0.00 -> 7.81 mm
- net /GPIO6: track 0.00 -> 6.33 mm
- net /GPIO5: track 0.00 -> 5.30 mm
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- added copper zone on In2.Cu, net +3V3
- added copper zone on B.Cu, net GND
- added copper zone on In1.Cu, net GND
- added copper zone on F.Cu, net VCC
Other:
- board text added: "10"
- board text added: "François Gervais 25 sept. 2021 rev 1.0"
- board text removed: "François Gervais 29 dec 2020 rev 1.0"
