File: hardware/project-esp32-c3-wroom-02-breakout.sch (KiCad schematic (older format))
At the start: 29 parts, among them J1 SM04B-SRSS-TB(LF)(SN), J2 Conn_01x08_Male, J3 Conn_01x08_Male, Q1 MUN5214DW1T1G, U1 XC6220B331MR, U2 ESP32-C3-WROOM-02-H4

Commit message: Annotate schematic
Parts:
- gave numbers to parts that had none: 12
Changed lines of the file:
@@
 USB_D-
 $Comp
-L Device:C_Small C?
+L Device:C_Small C5
 U 1 1 61C946D3
 P 4500 3850
-F 0 "C?" H 4592 3896 50  0000 L CNN
+F 0 "C5" H 4592 3896 50  0000 L CNN
 F 1 "22uF" H 4592 3805 50  0000 L CNN
 F 2 "Capacitor_SMD:C_0805_2012Metric_Pad1.18x1.45mm_HandSolder" H 4500 3850 50  0001 C CNN
@@
 	9700 3750 10350 3750
 $Comp
-L USB4105-GF-A:USB4105-GF-A J?
+L USB4105-GF-A:USB4105-GF-A J4
 U 1 1 61DFEFED
 P 8300 5400
-F 0 "J?" H 8300 6067 50  0000 C CNN
+F 0 "J4" H 8300 6067 50  0000 C CNN
 F 1 "USB4105-GF-A" H 8300 5976 50  0000 C CNN
 F 2 "GCT_USB4105-GF-A" H 8300 5400 50  0001 L BNN
@@
 $EndComp
 $Comp
-L power:GND #PWR?
+L power:GND #PWR05
 U 1 1 61E05717
 P 9400 5950
-F 0 "#PWR?" H 9400 5700 50  0001 C CNN
+F 0 "#PWR05" H 9400 5700 50  0001 C CNN
 F 1 "GND" H 9405 5777 50  0000 C CNN
 F 2 "" H 9400 5950 50  0001 C CNN
@@
 VBUS
 $Comp
-L Device:R_Small R?
+L Device:R_Small R8
 U 1 1 61E1A67C
 P 10500 4850
-F 0 "R?" H 10559 4896 50  0000 L CNN
+F 0 "R8" H 10559 4896 50  0000 L CNN
 F 1 "5.1k" H 10559 4805 50  0000 L CNN
 F 2 "Resistor_SMD:R_0603_1608Metric_Pad0.98x0.95mm_HandSolder" H 10500 4850 50  0001 C CNN
@@
 $EndComp
 $Comp
-L Device:R_Small R?
+L Device:R_Small R9
 U 1 1 61E1A682
 P 10800 4850
-F 0 "R?" H 10859 4896 50  0000 L CNN
+F 0 "R9" H 10859 4896 50  0000 L CNN
 F 1 "5.1k" H 10859 4805 50  0000 L CNN
 F 2 "Resistor_SMD:R_0603_1608Metric_Pad0.98x0.95mm_HandSolder" H 10800 4850 50  0001 C CNN
@@
 CC2
 $Comp
-L power:GND #PWR?
+L power:GND #PWR06
 U 1 1 61E409C2
 P 10800 5150
-F 0 "#PWR?" H 10800 4900 50  0001 C CNN
+F 0 "#PWR06" H 10800 4900 50  0001 C CNN
 F 1 "GND" H 10805 4977 50  0000 C CNN
 F 2 "" H 10800 5150 50  0001 C CNN
@@
 NoConn ~ 7200 5500
 $Comp
-L Device:R_Small R?
+L Device:R_Small R7
 U 1 1 61F4C1E9
 P 1500 1950
-F 0 "R?" H 1559 1996 50  0000 L CNN
+F 0 "R7" H 1559 1996 50  0000 L CNN
 F 1 "100k" H 1559 1905 50  0000 L CNN
 F 2 "Resistor_SMD:R_0603_1608Metric_Pad0.98x0.95mm_HandSolder" H 1500 1950 50  0001 C CNN
@@
 $EndComp
 $Comp
-L Device:Q_PMOS_DGS Q?
+L Device:Q_PMOS_DGS Q2
 U 1 1 61F4EE69
 P 2100 1200
-F 0 "Q?" H 2305 1246 50  0000 L CNN
+F 0 "Q2" H 2305 1246 50  0000 L CNN
 F 1 "Q_PMOS_DGS" H 2305 1155 50  0000 L CNN
 F 2 "SSM6J214FE-TE85L-F:SOT50P160X60-6N" H 2300 1300 50  0001 C CNN
@@
 $EndComp
 $Comp
-L power:+BATT #PWR?
+L power:+BATT #PWR03
 U 1 1 61F5D4F0
 P 2200 900
-F 0 "#PWR?" H 2200 750 50  0001 C CNN
+F 0 "#PWR03" H 2200 750 50  0001 C CNN
 F 1 "+BATT" H 2215 1073 50  0000 C CNN
 F 2 "" H 2200 900 50  0001 C CNN
@@
 VBAT
 $Comp
-L power:VBUS #PWR?
+L power:VBUS #PWR01
 U 1 1 61F93F0E
 P 1500 900
-F 0 "#PWR?" H 1500 750 50  0001 C CNN
+F 0 "#PWR01" H 1500 750 50  0001 C CNN
 F 1 "VBUS" H 1515 1073 50  0000 C CNN
 F 2 "" H 1500 900 50  0001 C CNN
@@
 $EndComp
 $Comp
-L power:GND #PWR?
+L power:GND #PWR02
 U 1 1 61F95635
 P 1500 2200
-F 0 "#PWR?" H 1500 1950 50  0001 C CNN
+F 0 "#PWR02" H 1500 1950 50  0001 C CNN
 F 1 "GND" H 1505 2027 50  0000 C CNN
 F 2 "" H 1500 2200 50  0001 C CNN
@@
 Alternative:\n‎RT9080-33GJ5‎
 $Comp
-L Device:D_Schottky D?
+L Device:D_Schottky D2
 U 1 1 61F47B46
 P 1850 1600
-F 0 "D?" H 1850 1383 50  0000 C CNN
+F 0 "D2" H 1850 1383 50  0000 C CNN
 F 1 "CUS10S30,H3F‎" H 1850 1474 50  0000 C CNN
 F 2 "CUS10S30,H3F:DIO_CUS520,H3F" H 1850 1600 50  0001 C CNN
@@
 USB_D+
 $Comp
-L Connector:TestPoint TP?
+L Connector:TestPoint TP1
 U 1 1 62261A96
 P 9550 5300
-F 0 "TP?" H 9608 5418 50  0000 L CNN
+F 0 "TP1" H 9608 5418 50  0000 L CNN
 F 1 "TestPoint" H 9608 5327 50  0000 L CNN
 F 2 "TestPoint:TestPoint_Pad_D1.0mm" H 9750 5300 50  0001 C CNN
@@
 $EndComp
 $Comp
-L Connector:TestPoint TP?
+L Connector:TestPoint TP2
 U 1 1 6226EE9C
 P 9550 5400
-F 0 "TP?" H 9492 5426 50  0000 R CNN
+F 0 "TP2" H 9492 5426 50  0000 R CNN
 F 1 "TestPoint" H 9492 5517 50  0000 R CNN
 F 2 "TestPoint:TestPoint_Pad_D1.0mm" H 9750 5400 50  0001 C CNN
@@
 	9100 5400 9550 5400
 $Comp
-L Connector:TestPoint TP?
+L Connector:TestPoint TP3
 U 1 1 6227B10D
 P 9550 5800
-F 0 "TP?" H 9608 5918 50  0000 L CNN
+F 0 "TP3" H 9608 5918 50  0000 L CNN
 F 1 "TestPoint" H 9608 5827 50  0000 L CNN
 F 2 "TestPoint:TestPoint_Pad_D1.0mm" H 9750 5800 50  0001 C CNN
@@
 	5050 5650 5050 5700
 $Comp
-L power:GND #PWR?
+L power:GND #PWR04
 U 1 1 62255EAE
 P 5050 5800
-F 0 "#PWR?" H 5050 5550 50  0001 C CNN
+F 0 "#PWR04" H 5050 5550 50  0001 C CNN
 F 1 "GND" H 5055 5627 50  0000 C CNN
 F 2 "" H 5050 5800 50  0001 C CNN
@@
 $EndComp
 $Comp
-L Mechanical:MountingHole_Pad H?
+L Mechanical:MountingHole_Pad H2
 U 1 1 62254682
 P 6000 5550
-F 0 "H?" H 6100 5599 50  0000 L CNN
+F 0 "H2" H 6100 5599 50  0000 L CNN
 F 1 "MountingHole_Pad" H 6100 5508 50  0000 L CNN
 F 2 "MountingHole:MountingHole_2.7mm_M2.5_ISO7380_Pad" H 6000 5550 50  0001 C CNN
@@
 $EndComp
 $Comp
-L Mechanical:MountingHole_Pad H?
+L Mechanical:MountingHole_Pad H1
 U 1 1 6225365F
 P 5050 5550
-F 0 "H?" H 5150 5599 50  0000 L CNN
+F 0 "H1" H 5150 5599 50  0000 L CNN
 F 1 "MountingHole_Pad" H 5150 5508 50  0000 L CNN
 F 2 "MountingHole:MountingHole_2.7mm_M2.5_ISO7380_Pad" H 5050 5550 50  0001 C CNN

Commit message: Change schottky footprint
Parts:
- D2: footprint CUS10S30,H3F:DIO_CUS520,H3F -> Diode_SMD:D_SOD-323_HandSoldering
Changed lines of the file:
@@
 F 0 "D2" H 1850 1383 50  0000 C CNN
 F 1 "CUS10S30,H3F‎" H 1850 1474 50  0000 C CNN
-F 2 "CUS10S30,H3F:DIO_CUS520,H3F" H 1850 1600 50  0001 C CNN
+F 2 "Diode_SMD:D_SOD-323_HandSoldering" H 1850 1600 50  0001 C CNN
 F 3 "~" H 1850 1600 50  0001 C CNN
 	1    1850 1600

Commit message: Change mounting hole to M2
Parts:
- H1, H2: footprint MountingHole:MountingHole_2.7mm_M2.5_ISO7380_Pad -> MountingHole:MountingHole_2.2mm_M2_ISO7380_Pad
Changed lines of the file:
@@
 F 0 "H2" H 6100 5599 50  0000 L CNN
 F 1 "MountingHole_Pad" H 6100 5508 50  0000 L CNN
-F 2 "MountingHole:MountingHole_2.7mm_M2.5_ISO7380_Pad" H 6000 5550 50  0001 C CNN
+F 2 "MountingHole:MountingHole_2.2mm_M2_ISO7380_Pad" H 6000 5550 50  0001 C CNN
 F 3 "~" H 6000 5550 50  0001 C CNN
 	1    6000 5550
@@
 F 0 "H1" H 5150 5599 50  0000 L CNN
 F 1 "MountingHole_Pad" H 5150 5508 50  0000 L CNN
-F 2 "MountingHole:MountingHole_2.7mm_M2.5_ISO7380_Pad" H 5050 5550 50  0001 C CNN
+F 2 "MountingHole:MountingHole_2.2mm_M2_ISO7380_Pad" H 5050 5550 50  0001 C CNN
 F 3 "~" H 5050 5550 50  0001 C CNN
 	1    5050 5550
